Commit message: Alles bis unterarm

File: install/robu/share/robu/urdf/example_robot.urdf.xacro (robot description, xacro)
@@ -17,10 +17,11 @@
         <parent link="world" />
         <child link="base" />
-        <origin  rpy="1.57 0 0" xyz="0 0 0" />
+        <origin  rpy="1.57 0 0" xyz="-3.5 0 0" />
     </joint>
     <link name="base">
         <visual>
-            <origin xyz="2 0 0" rpy="0 0 0"/>
+            <origin xyz="0.15 2.8 0" rpy="0 0 4.712"/>
             <geometry>
+                <mesh filename="package://robu/meshes/Basis.stl" scale="0.005 0.005 0.005"/>
                 <box size="5 0.1 3" />
             </geometry>
@@ -28,15 +29,16 @@
         </visual>
     </link>
-    <joint name="base_to_l3" type="revolute">
+    <joint name="base_to_l3" type="prismatic">
         <parent link="base" />
         <child link="l3" />
-        <origin  rpy="0 0 0" xyz="0 0.25 0" />
+        <origin  rpy="4.712 0 0" xyz="0 3 0" />
         <axis rpy="0 0 0" xyz="0 0 1" />
-        <limit effort="0.1" lower="-3.1" upper="3.1" velocity="0.2"/>
+        <limit effort="0.1" lower="-1.5" upper="1.5" velocity="0.2"/>
     </joint>
     <link name="l3">
         <visual>
-            <origin xyz="0.75 0 0" rpy="0 1.57 0"/>
+            <origin xyz="-0.025 0 0" rpy="1.5708 1.5708 0"/>
             <geometry>
+                <mesh filename="package://robu/meshes/Schulter.stl" scale="0.005 0.005 0.005"/>
                 <cylinder length="1.5" radius="0.04" />
             </geometry>
@@ -48,12 +50,13 @@
         <child link="l2" />
         <!-- <origin xyz="1 0 0" /> -->
-        <origin rpy="0 0 0" xyz="1.5 0 0" />
+        <origin rpy="0 0 0" xyz="0.56 0 0" />
         <axis rpy="0 0 0" xyz="0 0 1" />
-        <limit effort="0.1" lower="-3.1" upper="3.1" velocity="0.2"/>
+        <limit effort="0.1" lower="-1.65" upper="1.65" velocity="0.2"/>
     </joint>
     <link name="l2">
         <visual>
-            <origin xyz="0.75 0 0" rpy="0 1.57 0"/>
+            <origin xyz="4.38 0.055 -2.35" rpy="0 1.57 -1.57"/>
             <geometry>
+                <mesh filename="package://robu/meshes/Oberarm.stl" scale="0.005 0.005 0.005"/>
                 <cylinder length="1.5" radius="0.04" />
             </geometry>
@@ -64,12 +67,13 @@
         <parent link="l2" />
         <child link="l1" />
-        <origin rpy="0 0 0" xyz="1.5 0 0" />
+        <origin rpy="0 0 0" xyz="2.825 0 0.4" />
         <axis rpy="0 0 0" xyz="0 0 1" />
-        <limit effort="0.1" lower="-3.1" upper="3.1" velocity="0.2"/>
+        <limit effort="0.1" lower="-2.5" upper="2.5" velocity="0.2"/>
     </joint>
     <link name="l1">
         <visual>
-            <origin xyz="0.5 0 0" rpy="0 1.57 0"/>
+            <origin xyz="1.143 -0.06 0" rpy="0 1.57 -1.57"/>
             <geometry>
+                <mesh filename="package://robu/meshes/Unterarm.stl" scale="0.005 0.005 0.005"/>
                 <cylinder length="1" radius="0.04" />
             </geometry>
@@ -80,5 +84,5 @@
         <parent link="l1" />
         <child link="grip" />
-        <origin rpy="0 0 0" xyz="1 0 0" />
+        <origin rpy="0 0 0" xyz="2.48 -0.03 -0.2" />
         <axis rpy="0 0 0" xyz="0 0 1" />
         <limit effort="0.1" lower="-3.1" upper="3.1" velocity="0.2"/>

Commit message: Fertig

File: install/robu/share/robu/urdf/example_robot.urdf.xacro (robot description, xacro)
@@ -90,6 +90,7 @@
     <link name="grip">
         <visual>
-            <origin xyz="0.25 0 0"/>
+            <origin xyz="-0.1 0.2 -0.52" rpy="0 1.5708 0"/>
             <geometry>
+                <mesh filename="package://robu/meshes/Hand.stl" scale="0.005 0.005 0.005"/>
                 <box size="0.5 0.5 0.05" />
             </geometry>

Commit message: FERRTIIIGGGG

File: install/robu/share/robu/urdf/example_robot.urdf.xacro (robot description, xacro)
@@ -28,4 +28,10 @@
             <material name="grey" />
         </visual>
+        <collision>
+            <origin xyz="0.15 2.875 0" rpy="0 0 0"/>
+            <geometry>
+                <box size="2 5.75 1.8"/>
+            </geometry>
+        </collision>
     </link>
     <joint name="base_to_l3" type="prismatic">
@@ -63,4 +69,10 @@
             <material name="orange" />
         </visual>
+        <collision>
+            <origin xyz="1.45 -0.01 0" rpy="0 0 0"/>
+            <geometry>
+                <box size="3.5 0.75 1.5"/>
+            </geometry>
+        </collision>
     </link>
     <joint name="l2_to_l1" type="revolute">
@@ -80,4 +92,10 @@
             <material name="orange" />
         </visual>
+        <collision>
+            <origin xyz="1.2 0 0" rpy="0 0 0"/>
+            <geometry>
+                <box size="3 0.7 0.4"/>
+            </geometry>
+        </collision>
     </link>
     <joint name="l1_to_grip" type="revolute">
@@ -97,18 +115,10 @@
             <material name="white" />
         </visual>
-    </link>
-    <joint name="world_to_camera" type="fixed">
-        <parent link="world" />
-        <child link="camera" />
-        <origin  rpy="-2 0 2.5" xyz="4 1 2" />
-    </joint>
-    <link name="camera">
-        <visual>
-            <origin xyz="0 0 -0.2"/>
+        <collision>
+            <origin xyz="0 0 -0.3" rpy="0 0 0"/>
             <geometry>
-                <box size="0.2 0.2 0.4" />
+                <box size="0.4 0.6 0.6"/>
             </geometry>
-            <material name="blue" />
-        </visual>
+        </collision>
     </link>
 </robot>
